Commit message: Updated some mismatched params for this platform

File: description/urdf/diffbot_description.urdf.xacro (robot description, xacro)
@@ -10,5 +10,5 @@
   <xacro:property name="wheel_mass" value="0.3" /> <!-- arbitrary value for wheel mass -->
   <xacro:property name="wheel_len" value="0.020" />
-  <xacro:property name="wheel_radius" value="0.0175" />
+  <xacro:property name="wheel_radius" value="0.0215" />
   <xacro:property name="imu_height" value="0.04" /> <!-- Height of IMU below top plate -->
   <!-- Base Link -->

Commit message: Fixed some behaviour. Adjusted urdf

File: description/urdf/diffbot_description.urdf.xacro (robot description, xacro)
@@ -6,14 +6,14 @@
   <xacro:property name="base_mass" value="0.3" /> <!-- arbitrary value for base mass -->
   <xacro:property name="base_width" value="0.14" />
-  <xacro:property name="base_length" value="0.14" />
-  <xacro:property name="base_height" value="0.05" />
-  <xacro:property name="wheel_mass" value="0.3" /> <!-- arbitrary value for wheel mass -->
+  <xacro:property name="base_length" value="0.135" />
+  <xacro:property name="base_height" value="0.061" />
+  <xacro:property name="wheel_mass" value="0.05" /> <!-- arbitrary value for wheel mass -->
   <xacro:property name="wheel_len" value="0.020" />
   <xacro:property name="wheel_radius" value="0.0215" />
-  <xacro:property name="imu_height" value="0.04" /> <!-- Height of IMU below top plate -->
+  <xacro:property name="offset" value="0.0425" />
   <!-- Base Link -->
   <link name="${prefix}base_link">
     <collision>
-      <origin xyz="0 0 0" rpy="0 0 0"/>
+      <origin xyz="${offset} 0 0" rpy="0 0 0"/>
       <geometry>
         <box size="${base_width} ${base_length} ${base_height}"/>
@@ -21,5 +21,5 @@
     </collision>
     <visual>
-      <origin xyz="0 0 ${base_height/2}" rpy="0 0 0"/>
+      <origin xyz="${offset} 0 ${base_height/2}" rpy="0 0 0"/>
       <geometry>
         <box size="${base_width} ${base_length} ${base_height}"/>
@@ -28,5 +28,5 @@
     </visual>
     <inertial>
-      <origin xyz="0 0 0" rpy="0 0 0"/>
+      <origin xyz="${offset} 0 0" rpy="0 0 0"/>
       <mass value="${base_mass}"/>
       <inertia
@@ -36,12 +36,4 @@
       </inertial>
     </link>
-    <!-- left wheel Joint -->
-    <joint name="${prefix}left_wheel_joint" type="continuous">
-      <parent link="${prefix}base_link"/>
-      <child link="${prefix}left_wheel"/>
-      <origin xyz="0.02 ${base_width/2} 0" rpy="0 0 0"/>
-      <axis xyz="0 1 0"/>
-      <dynamics damping="0.2"/>
-    </joint>
     <joint name="${prefix}base_footprint_joint" type="fixed">
       <parent link="${prefix}base_link"/>
@@ -51,4 +43,12 @@
     <link name="base_footprint">
     </link>
+    <!-- left wheel Joint -->
+    <joint name="${prefix}left_wheel_joint" type="continuous">
+      <parent link="${prefix}base_link"/>
+      <child link="${prefix}left_wheel"/>
+      <origin xyz="0 ${0.17/2} 0" rpy="0 0 0"/>
+      <axis xyz="0 1 0"/>
+      <dynamics damping="0.2"/>
+    </joint>
     <!-- left wheel Link -->
     <link name="${prefix}left_wheel">
@@ -79,5 +79,5 @@
       <parent link="${prefix}base_link"/>
       <child link="${prefix}right_wheel"/>
-      <origin xyz="0.02 -${base_width/2} 0" rpy="0 0 0"/>
+      <origin xyz="0 -${0.17/2} 0" rpy="0 0 0"/>
       <axis xyz="0 1 0"/>
       <dynamics damping="0.2"/>
@@ -120,5 +120,5 @@
       <parent link="${prefix}base_link"/>
       <child link="${prefix}imu_link"/>
-      <origin xyz="-0.02 0.01 ${base_height - imu_height}" rpy="0 0 ${PI}"/>
+      <origin xyz="${-0.0225+offset} 0.01 ${base_height + 0.02}" rpy="0 0 ${PI}"/>
     </joint>
           <!-- Lidar Sensor -->
@@ -135,5 +135,5 @@
       <parent link="${prefix}base_link"/>
       <child link="${prefix}laser"/>
-      <origin xyz="0 0 ${base_height + 0.04}" rpy="0 0 ${PI}"/>
+      <origin xyz="${-0.0225+offset} 0 ${base_height + 0.04}" rpy="0 0 ${PI}"/>
     </joint>
     <!-- Camera -->
@@ -142,5 +142,5 @@
         <origin xyz="0 0 0" rpy="0 0 0"/>
         <geometry>
-          <box size="0.01 0.025 0.025"/>
+          <box size="0.005 0.035 0.034"/>
         </geometry>
         <material name="green"/>
@@ -150,5 +150,5 @@
       <parent link="${prefix}base_link"/>
       <child link="${prefix}camera_link"/>
-      <origin xyz="0.08 0 ${base_height - imu_height}" rpy="0 0 0"/>
+      <origin xyz="${0.0635+offset} 0 ${base_height - 0.0177}" rpy="0 0 0"/>
     </joint>
     <link name="${prefix}camera_link_optical"></link>
